File: 1.KiCAD/Pixel.Combs/Pixel.Combs.kicad_pcb (KiCad board)
At the start: 2 copper layers, 247 x 170 mm, 170 parts

Commit message: Added a second design of the Steel Vessel
Parts:
- removed the ? at (100.0, 148.3)
- removed the ? at (65.0, 113.3)
- removed the ? at (173.2, 173.0)
- removed the ? at (256.7, 173.0)
- removed the ? at (89.7, 123.5)
- removed the ? at (123.7, 173.0)
- removed the ? at (183.5, 148.3)
- removed the ? at (40.2, 123.5)
- removed the ? at (123.7, 123.5)
- removed the ? at (148.5, 183.3)
- removed the ? at (173.2, 123.5)
- removed the ? at (207.2, 123.5)
- removed the ? at (267.0, 148.3)
- removed the ? at (232.0, 113.3)
- removed the ? at (148.5, 113.3)
- removed the ? at (113.5, 148.3)
- removed the ? at (197.0, 148.3)
- removed the ? at (207.2, 173.0)
- removed the ? at (89.7, 173.0)
- removed the ? at (40.2, 173.0)
- removed the ? at (30.0, 148.3)
- removed the ? at (65.0, 183.3)
- removed the ? at (256.7, 123.5)
- removed the ? at (232.0, 183.3)
- removed the G*** at (219.6, 178.2)
- removed the G*** at (52.6, 178.2)
- removed the G*** at (136.1, 178.2)
- removed the REF** at (65.0, 148.3)
- removed the REF** at (232.0, 148.3)
- removed the REF** at (148.5, 148.3)
- removed the REF**1 at (75.0, 148.3)
- removed the REF**10 at (153.5, 139.6)
- removed the REF**11 at (163.5, 139.6)
- removed the REF**12 at (252.0, 148.3)
- removed the REF**13 at (138.5, 131.0)
- removed the REF**14 at (148.5, 131.0)
- removed the REF**15 at (158.5, 131.0)
- removed the REF**18 at (237.0, 157.0)
- removed the REF**19 at (60.0, 139.6)
- removed the REF**2 at (85.0, 148.3)
- removed the REF**20 at (70.0, 139.6)
- removed the REF**21 at (80.0, 139.6)
- removed the REF**22 at (247.0, 157.0)
- removed the REF**23 at (55.0, 131.0)
- removed the REF**24 at (65.0, 131.0)
- removed the REF**25 at (75.0, 131.0)
- removed the REF**29 at (242.0, 165.6)
- removed the REF**3 at (158.5, 148.3)
- removed the REF**30 at (153.5, 157.0)
- removed the REF**31 at (55.0, 148.3)
- removed the REF**32 at (45.0, 148.3)
- removed the REF**33 at (163.5, 157.0)
- removed the REF**35 at (60.0, 157.0)
- removed the REF**36 at (50.0, 157.0)
- removed the REF**38 at (158.5, 165.6)
- removed the REF**39 at (65.0, 165.6)
- removed the REF**4 at (70.0, 157.0)
- removed the REF**40 at (55.0, 165.6)
- removed the REF**49 at (50.0, 139.6)
- removed the REF**5 at (80.0, 157.0)
- removed the REF**50 at (128.5, 148.3)
- removed the REF**53 at (133.5, 139.6)
- removed the REF**59 at (227.0, 139.6)
- removed the REF**6 at (168.5, 148.3)
- removed the REF**60 at (237.0, 139.6)
- removed the REF**61 at (247.0, 139.6)
- removed the REF**63 at (222.0, 131.0)
- removed the REF**64 at (138.5, 148.3)
- removed the REF**65 at (232.0, 131.0)
- removed the REF**66 at (242.0, 131.0)
- removed the REF**67 at (143.5, 157.0)
- removed the REF**68 at (133.5, 157.0)
- removed the REF**7 at (242.0, 148.3)
- removed the REF**71 at (138.5, 165.6)
- removed the REF**75 at (222.0, 148.3)
- removed the REF**76 at (212.0, 148.3)
- removed the REF**79 at (227.0, 157.0)
- removed the REF**8 at (75.0, 165.6)
- removed the REF**80 at (148.5, 165.6)
- removed the REF**81 at (217.0, 157.0)
- removed the REF**84 at (232.0, 165.6)
- removed the REF**85 at (222.0, 165.6)
- removed the REF**9 at (143.5, 139.6)
- removed the REF**91 at (212.0, 148.3)
- removed the REF**94 at (217.0, 139.6)
Routing:
- net (no net): track 537.8 -> 268.9 mm, vias 194 -> 97
Other:
- board size 247 x 170 mm -> 247 x 80 mm

Commit message: Major changes to readout design
Parts:
- removed ? (x24): , 
- removed G***: Designed by Alfredo Barajas Enriquez, LOGO
- removed G*** (x2): LOGO, LOGO
Other:
- board size 247 x 80 mm -> 245 x 78 mm
- board text added: "May 2023 Alfredo Barajas Enriquez"

Commit message: Updated texts on files
Other:
- board text added: "Complex Dot Hexagon ::: May 2023 Alfredo Barajas Enriquez"
- board text added: "Complex Hexagon Full ::: May 2023 Alfredo Barajas Enriquez"
- board text added: "Simple Hexagon Pixel ::: May 2023 Alfredo Barajas Enriquez"
- board text removed: "May 2023 Alfredo Barajas Enriquez"
Changed lines of the file:
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@@
   (gr_circle (center 64.955 58.295) (end 99.955 58.295)
     (stroke (width 10) (type solid)) (fill none) (layer "F.Mask"))
-  (gr_circle (center 64.953889 148.295589) (end 94.953889 148.295589)
-    (stroke (width 0.1) (type solid)) (fill solid) (layer "F.Mask"))
-  (gr_circle (center 148.458652 148.295652) (end 188.458652 148.295652)
-    (stroke (width 1) (type solid)) (fill solid) (layer "F.Mask"))
-  (gr_circle (center 64.953889 148.295589) (end 99.953889 148.295589)
-    (stroke (width 10) (type solid)) (fill none) (layer "F.Mask"))
-  (gr_circle (center 231.963511 148.295745) (end 271.963511 148.295745)
-    (stroke (width 1) (type solid)) (fill solid) (layer "F.Mask"))
   (gr_circle (center 231.964622 58.295156) (end 271.964622 58.295156)
     (stroke (width 1) (type solid)) (fill solid) (layer "F.Mask"))
@@
   (gr_circle (center 216.964622 32.315156) (end 217.064622 32.315156)
     (stroke (width 0.1) (type solid)) (fill none) (layer "User.8"))
-  (gr_line locked (start 64.953889 148.295589) (end 231.963889 148.295589)
-    (stroke (width 0.1) (type default)) (layer "User.8"))
   (gr_circle (center 148.459763 58.295063) (end 148.559763 58.295063)
     (stroke (width 0.1) (type solid)) (fill solid) (layer "User.8"))
@@
   (gr_circle (center 89.955 66.955) (end 90.055 66.955)
     (stroke (width 0.1) (type solid)) (fill solid) (layer "User.8"))
-  (gr_line locked (start 148.46 58.295) (end 148.46 148.295)
-    (stroke (width 0.1) (type default)) (layer "User.8"))
   (gr_arc (start 123.711026 33.546326) (mid 135.065837 25.959259) (end 148.459763 23.295063)
     (stroke (width 0.2) (type solid)) (layer "User.8"))
@@
   (gr_circle (center 148.459763 58.295063) (end 183.459763 58.295063)
     (stroke (width 0.2) (type solid)) (fill none) (layer "User.8"))
-  (gr_text "May 2023\nAlfredo Barajas Enriquez\n" (at 241.655 88.375) (layer "B.SilkS")
+  (gr_text "Complex Hexagon Full ::: May 2023\nAlfredo Barajas Enriquez\n" (at 244.925 89.355) (layer "B.SilkS")
     (effects (font (size 1 1) (thickness 0.15)) (justify left bottom mirror))
   )
-  (gr_text "May 2023\nAlfredo Barajas Enriquez\n" (at 74.625 88.405) (layer "B.SilkS")
+  (gr_text "Simple Hexagon Pixel ::: May 2023\nAlfredo Barajas Enriquez" (at 76.87 89.57) (layer "B.SilkS")
     (effects (font (size 1 1) (thickness 0.15)) (justify left bottom mirror))
   )
-  (gr_text "May 2023\nAlfredo Barajas Enriquez\n" (at 158.1 88.385) (layer "B.SilkS")
+  (gr_text "Complex Dot Hexagon ::: May 2023\nAlfredo Barajas Enriquez\n" (at 161.86 89.17) (layer "B.SilkS")
     (effects (font (size 1 1) (thickness 0.15)) (justify left bottom mirror))
   )
