File: Channel.Tester/KiCAD/channel.tester.kicad_pcb (KiCad board)
At the start: 2 copper layers, 78 x 78 mm, 19 parts

Commit message: Minor Fixes
Parts:
- added G***: LOGO, LOGO, B.Cu at (64.0, 85.7)
Other:
- board text added: "Channel Tester ::: May 2023 Alfredo Barajas Enriquez"
- board text removed: "SAQ-Channel Tester ::: May 2023 Alfredo Barajas Enriquez"
