File: Modular.Pixel.Combs/5.Pixel.Comb.Base.Empty/KiCAD/Pixel.Comb.Base.kicad_pcb (KiCad board)
At the start: 2 copper layers, 78 x 78 mm, 0 parts

Commit message: Minor Fixes
Parts:
- added G***: LOGO, LOGO, B.Cu at (68.1, 86.4)
